File: avrisp-mkII-clone/avrisp-mkII-clone.kicad_pcb (KiCad board)
At the start: 2 copper layers, 0 parts

Commit message: update project file
Parts:
- added C1: 100n, Capacitor_SMD:C_0805_2012Metric_Pad1.15x1.40mm_HandSolder, B.Cu at (109.2, 88.9)
- added C10: 100n, Capacitor_SMD:C_0805_2012Metric_Pad1.15x1.40mm_HandSolder, F.Cu at (149.5, 104.8)
- added C2: 33p, Capacitor_SMD:C_0805_2012Metric_Pad1.15x1.40mm_HandSolder, F.Cu at (106.0, 132.7)
- added C3: 33p, Capacitor_SMD:C_0805_2012Metric_Pad1.15x1.40mm_HandSolder, F.Cu at (111.1, 132.7)
- added C4: 1u, Capacitor_SMD:C_0805_2012Metric_Pad1.15x1.40mm_HandSolder, F.Cu at (109.9, 101.6)
- added C5: 100n, Capacitor_SMD:C_0805_2012Metric_Pad1.15x1.40mm_HandSolder, F.Cu at (116.0, 101.6)
- added C6: 10u, Capacitor_Tantalum_SMD:CP_EIA-7343-15_Kemet-W_Pad2.25x2.55mm_HandSolder, F.Cu at (94.0, 104.1)
- added C7: 100n, Capacitor_SMD:C_0805_2012Metric_Pad1.15x1.40mm_HandSolder, F.Cu at (149.2, 116.8)
- added C8: 10u, Capacitor_Tantalum_SMD:CP_EIA-7343-15_Kemet-W_Pad2.25x2.55mm_HandSolder, F.Cu at (148.6, 91.4)
- added C9: 10u, Capacitor_Tantalum_SMD:CP_EIA-7343-15_Kemet-W_Pad2.25x2.55mm_HandSolder, F.Cu at (128.9, 91.4)
- added D1: 1N4148W, Diode_SMD:D_SOD-123, F.Cu at (104.8, 100.3)
- added D2: PWR, LED_THT:LED_D3.0mm, F.Cu at (149.9, 130.8)
- added D3: PRG, LED_THT:LED_D3.0mm, F.Cu at (142.2, 130.8)
- added FB1: 050, Resistor_SMD:R_1206_3216Metric_Pad1.42x1.75mm_HandSolder, F.Cu at (119.4, 94.6)
- added J1: usb micro, Connector_USB:USB_Micro-B_Molex_47346-0001, F.Cu at (91.4, 119.4)
- added J2: AVR-PDI-6, Connector_IDC:IDC-Header_2x03_P2.54mm_Vertical, F.Cu at (179.7, 106.7)
- added J3: AVR-TPI-6, Connector_IDC:IDC-Header_2x03_P2.54mm_Vertical, F.Cu at (190.5, 106.7)
- added JP1: 5V/3.3V, Connector_PinHeader_2.54mm:PinHeader_1x03_P2.54mm_Vertical, F.Cu at (161.3, 97.2)
- added JP2: prg/cir, Connector_PinHeader_2.54mm:PinHeader_1x03_P2.54mm_Vertical, F.Cu at (179.1, 94.6)
- added M1: MountingHole_2.2mm_M2_DIN965, MountingHole:MountingHole_2.2mm_M2_DIN965, F.Cu at (91.4, 86.4)
- added M2: MountingHole_2.2mm_M2_DIN965, MountingHole:MountingHole_2.2mm_M2_DIN965, F.Cu at (200.7, 86.4)
- added M3: MountingHole_2.2mm_M2_DIN965, MountingHole:MountingHole_2.2mm_M2_DIN965, F.Cu at (200.7, 134.6)
- added M4: MountingHole_2.2mm_M2_DIN965, MountingHole:MountingHole_2.2mm_M2_DIN965, F.Cu at (91.4, 134.6)
- added R1: 10k, Resistor_SMD:R_0805_2012Metric_Pad1.15x1.40mm_HandSolder, B.Cu at (109.2, 92.7)
- added R2: 1k, Resistor_SMD:R_0805_2012Metric_Pad1.15x1.40mm_HandSolder, F.Cu at (137.2, 113.0)
- added R3: 470R, Resistor_SMD:R_0805_2012Metric_Pad1.15x1.40mm_HandSolder, B.Cu at (152.4, 125.7)
- added R4: 470R, Resistor_SMD:R_0805_2012Metric_Pad1.15x1.40mm_HandSolder, B.Cu at (139.7, 126.0)
- added R5: 470R, Resistor_SMD:R_0805_2012Metric_Pad1.15x1.40mm_HandSolder, F.Cu at (137.2, 102.9)
- added R6: 470R, Resistor_SMD:R_0805_2012Metric_Pad1.15x1.40mm_HandSolder, F.Cu at (137.2, 121.3)
- added R7: 470R, Resistor_SMD:R_0805_2012Metric_Pad1.15x1.40mm_HandSolder, F.Cu at (137.2, 117.5)
- added REF**: OSHW-Logo2_14.6x12mm_SilkScreen, Symbol:OSHW-Logo2_14.6x12mm_SilkScreen, F.Cu at (162.6, 129.5)
- added SW1: reset, Button_Switch_THT:SW_PUSH_6mm_H5mm, F.Cu at (97.8, 88.9)
- added SW2: PRG, Button_Switch_THT:SW_PUSH_6mm_H5mm, F.Cu at (125.7, 128.3)
- added U1: AT90USB162-16AU, Package_QFP:TQFP-32_7x7mm_P0.8mm, F.Cu at (116.8, 112.4)
- added U2: LM1117-3.3, Package_TO_SOT_SMD:SOT-223, F.Cu at (138.9, 94.7)
- added U3: MAX3002EUP, Package_SO:TSSOP-20_4.4x6.5mm_P0.65mm, F.Cu at (149.2, 111.1)
- added U4: AVR-ISP10, Connector_IDC:IDC-Header_2x05_P2.54mm_Vertical, F.Cu at (168.9, 106.7)
- added Y1: 16 MHz, Crystal:Crystal_SMD_HC49-SD_HandSoldering, F.Cu at (108.6, 126.4)
Routing:
- net GND: track 0.00 -> 321.5 mm, vias 0 -> 1
- net +5V: track 0.00 -> 149.4 mm, vias 0 -> 3
- net Net-(C10-Pad2): track 0.00 -> 47.9 mm
- net Net-(R2-Pad2): track 0.00 -> 43.9 mm, vias 0 -> 2
- net Net-(C8-Pad1): track 0.00 -> 43.5 mm
- net Net-(C1-Pad2): track 0.00 -> 42.6 mm
- net /DATA: track 0.00 -> 41.8 mm, vias 0 -> 1
- net Net-(R3-Pad1): track 0.00 -> 40.5 mm, vias 0 -> 1
- net /CLK: track 0.00 -> 40.3 mm
- net /RESET: track 0.00 -> 40.2 mm
- net Net-(R5-Pad2): track 0.00 -> 37.8 mm
- net VSS: track 0.00 -> 35.7 mm
- net Net-(C9-Pad1): track 0.00 -> 33.5 mm
- net Net-(U1-Pad17): track 0.00 -> 32.6 mm
- net Net-(U1-Pad16): track 0.00 -> 31.2 mm
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- added copper zone on F.Cu, net GND
Other:
- board outline added: 114.3 x 53.3 mm
- net class Default: trace_width 0.25 -> 0.4
- board text added: "5V/3.3V"
- board text added: "AVRISP MKII clone License: MIT by SQ7EQE rev.: 1.0, 2020"
- board text added: "AVRISP MKII clone programmer firmware: lufa"
- board text added: "ISP10"
- board text added: "PDI"
- board text added: "PRG"
- board text added: "PRG/CIRCUIT"
- board text added: "PWR"
- board text added: "RESET"
- board text added: "TPI"
- board text added: "https://majsterklepka.github.io"
